File: Hardware/Version_2/ELA_V2/ELA_V2.sch (KiCad schematic (older format))
At the start: 26 parts

Commit message: simplificacion de software
Parts:
- added AE1: Antenna, symbol Device:Antenna
- gave numbers to parts that had none: 26
Connections:
- net Vbatt: no longer F1.1, J3.1 (Pin_1), U4.8 (IN)
- net at U6.34 (ANTENNA): now also AE1.1 (A)
- net Vpan: no longer names the net of D1.1 (K), D2.2 (A), J1.2 (Pin_2)
- new net: F1.1, J3.1 (Pin_1), U4.8 (IN)
- no-connect marks 0 -> 38
Other:
- moved on the sheet: C3, C4, C5, C6, C7, D2, F1, J3, J5, J6, R2, U1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
